Commit message: valet_car 외형을 실차 메시로 교체 (Prius Hybrid, CC0)
박스 조합 외형을 실제 차량 메시로 바꿨다. 표준 방식대로
**visual 만 메시, collision 은 박스 6개**를 유지한다. 물리는 박스로 빠르고
안정적으로 풀고 눈에 보이는 것만 메시로 한다.

제원(전장 4.50 / 전폭 1.90 / 축거 2.50 / 최소회전반경 3.5704), 조인트,
ros2_control, 라이다 위치는 하나도 안 건드렸다. Nav2 와 맵 패키지 정합성도 그대로다.

## 원본과 제원이 달라 메시를 변형했다

              전장    전폭   축거    바퀴반경
  Prius      4.618   2.012  2.865   0.305
  valet_car  4.50    1.90   2.50    0.33

균일 스케일로는 축거가 안 맞아 바퀴가 휠아치에서 15 cm 어긋난다.
tools/fit_car_mesh.py 가 길이축을 구간별 선형 리매핑 한다.

  앞 오버행 x1.170    축간 x0.873    뒤 오버행 x1.112
  폭 x0.944          높이 x0.794

높이를 0.794 로 줄인 건 지붕이 1.34 m 여야 하기 때문이다. 라이다가 1.42 m 에
있고 그보다 지붕이 낮아야 360 도가 안 가린다.

결과: 전장 4.500 / 전폭 1.900 / 높이 0.240~1.340 — 목표와 정확히 일치.

## 성능 손해 없음

메시가 1680 면밖에 안 돼서 llvmpipe 로도 부담이 없다.

               RTF     라이다 유효 프레임   평균 빔
  박스 외형    1.000        100 %          427/720
  메시 외형    1.002        100 %          427/720

스모크 테스트 8/8 통과 (메시 적용 후 재측정):

  A. /scan       40 프레임 중 유효 40 (100%), 평균 427 빔, 최대 29.5 m
  C. 전진 8 s     이동 7.99 m
  D. 최소회전반경  실측 R = 3.47 m
  E. Ackermann   좌 40.18 / 우 29.95 (차 10.23 deg)
  F. 후진 5 s     -2.50 m
  H. 각속도 클램프 요청 2.0 -> 실측 0.252

## parking_world.launch.py: GZ_SIM_RESOURCE_PATH 를 Set -> Append

Set 으로 덮어쓰고 있어서, 다른 패키지가 ament 환경 훅으로 등록한 경로가
지워졌다. 그 탓에 로봇 패키지의 package://valet_robot/meshes/*.obj 를
Gazebo 가 못 찾았다 (Unable to find file[model://valet_robot/meshes/body.obj]).
AppendEnvironmentVariable 로 바꿔 해결.

## 추가

* meshes/                body.obj (1000 정점 / 1680 면), wheel.obj, mtl, 텍스처
* meshes/README.md       출처·라이선스·변형 방법·재생성 절차
* tools/fit_car_mesh.py  원본 OBJ 를 우리 제원에 맞춰 분리·변형
* tools/preview_model.py 메시 렌더링 지원 추가
* hooks/valet_robot.dsv.in  GZ_SIM_RESOURCE_PATH 에 share 등록
* mesh:=false 인자        박스 조합 외형으로 되돌리기 (메시 없이 확인할 때)

원본: Gazebo Fuel OpenRobotics/Prius Hybrid, 저자 Ian Chen, CC0 1.0 퍼블릭 도메인.
CC0 라 표기 의무는 없지만 meshes/README.md 에 출처를 남겼다.

File: src/valet_robot/urdf/body.xacro (robot description, xacro)
@@ -8,11 +8,13 @@
      ========================================================================== -->
 <robot xmlns:xacro="http://www.ros.org/wiki/xacro">
-  <!-- 충돌 박스 하나 = 같은 크기의 visual + collision -->
-  <xacro:macro name="body_box" params="name x y z sx sy sz material collision:=true">
-    <visual name="${name}_vis">
-      <origin xyz="${x} ${y} ${z}" rpy="0 0 0"/>
-      <geometry><box size="${sx} ${sy} ${sz}"/></geometry>
-      <material name="${material}"/>
-    </visual>
+  <!-- 박스 하나. visual 은 mesh 모드에서 끌 수 있다 -->
+  <xacro:macro name="body_box" params="name x y z sx sy sz material collision:=true visual:=true">
+    <xacro:if value="${visual}">
+      <visual name="${name}_vis">
+        <origin xyz="${x} ${y} ${z}" rpy="0 0 0"/>
+        <geometry><box size="${sx} ${sy} ${sz}"/></geometry>
+        <material name="${material}"/>
+      </visual>
+    </xacro:if>
     <xacro:if value="${collision}">
       <collision name="${name}_col">
@@ -44,60 +46,73 @@
   </xacro:macro>
   <!-- ===================== 차체 전체 ===================== -->
-  <xacro:macro name="car_body">
+  <xacro:macro name="car_body" params="use_mesh:=true">
+    <!-- === 외형: 메시 (실차 Prius 를 우리 제원에 맞춰 변형) === -->
+    <xacro:if value="${use_mesh}">
+      <visual name="body_mesh_vis">
+        <origin xyz="0 0 ${-base_z}" rpy="0 0 0"/>
+        <geometry>
+          <mesh filename="package://valet_robot/meshes/body.obj"/>
+        </geometry>
+      </visual>
+    </xacro:if>
     <!-- 하부: 플로어팬(축 사이만) + 앞뒤 범퍼. 사이 빈 공간이 휠아치 -->
     <xacro:body_box name="floor_pan" x="0" y="0" z="${pan_cz}"
                     sx="${pan_len}" sy="${pan_w}" sz="${pan_h}"
-                    material="valet_body"/>
+                    material="valet_body" visual="${not use_mesh}"/>
     <xacro:body_box name="bumper_f" x="${fascia_cx}" y="0" z="${pan_cz}"
                     sx="${fascia_len}" sy="${fascia_w}" sz="${pan_h}"
-                    material="valet_body"/>
+                    material="valet_body" visual="${not use_mesh}"/>
     <xacro:body_box name="bumper_r" x="${-fascia_cx}" y="0" z="${pan_cz}"
                     sx="${fascia_len}" sy="${fascia_w}" sz="${pan_h}"
-                    material="valet_body"/>
+                    material="valet_body" visual="${not use_mesh}"/>
     <!-- 벨트라인. 캐빈/후방(높음) + 보닛부(낮음) 로 나눠 앞머리를 낮춘다.
          둘을 합쳐 전장 4.50 x 전폭 1.90 이 나온다. -->
     <xacro:body_box name="belt_rear" x="${beltr_cx}" y="0" z="${beltr_cz}"
                     sx="${beltr_len}" sy="${body_width}" sz="${beltr_h}"
-                    material="valet_body"/>
+                    material="valet_body" visual="${not use_mesh}"/>
     <xacro:body_box name="belt_front" x="${beltf_cx}" y="0" z="${beltf_cz}"
                     sx="${beltf_len}" sy="${body_width}" sz="${beltf_h}"
-                    material="valet_body"/>
+                    material="valet_body" visual="${not use_mesh}"/>
     <!-- 보닛(경사판) / 트렁크 리드 -->
-    <visual name="hood_vis">
-      <origin xyz="${hood_cx} 0 ${hood_cz}" rpy="0 ${hood_pitch} 0"/>
-      <geometry><box size="${hood_len} ${lid_w} ${lid_h}"/></geometry>
-      <material name="valet_body"/>
-    </visual>
+    <xacro:unless value="${use_mesh}">
+      <visual name="hood_vis">
+        <origin xyz="${hood_cx} 0 ${hood_cz}" rpy="0 ${hood_pitch} 0"/>
+        <geometry><box size="${hood_len} ${lid_w} ${lid_h}"/></geometry>
+        <material name="valet_body"/>
+      </visual>
+    </xacro:unless>
     <xacro:body_box name="trunk" x="${trunk_cx}" y="0" z="${lid_cz}"
                     sx="${trunk_len}" sy="${lid_w}" sz="${lid_h}"
-                    material="valet_body" collision="false"/>
+                    material="valet_body" collision="false" visual="${not use_mesh}"/>
     <!-- 캐빈(그린하우스) + 루프 -->
     <xacro:body_box name="cabin" x="${cabin_cx}" y="0" z="${cabin_cz}"
                     sx="${cabin_len}" sy="${cabin_w}" sz="${cabin_h}"
-                    material="valet_glass"/>
+                    material="valet_glass" visual="${not use_mesh}"/>
     <xacro:body_box name="roof" x="${cabin_cx}" y="0" z="${roof_cz}"
                     sx="1.30" sy="1.68" sz="0.04"
-                    material="valet_body" collision="false"/>
-    <!-- 앞유리 / 뒷유리 (기울어진 판) -->
-    <xacro:glass_panel name="windshield" x="0.60"  z="0.81" plen="0.68" pitch="0.491"/>
-    <xacro:glass_panel name="rearglass"  x="-1.085" z="0.82" plen="0.41" pitch="-0.838"/>
-    <!-- 센서 포드 (지붕 위) -->
-    <visual name="sensor_pod_vis">
-      <origin xyz="0 0 ${pod_cz}" rpy="0 0 0"/>
-      <geometry><cylinder radius="0.10" length="0.05"/></geometry>
-      <material name="valet_metal"/>
-    </visual>
-    <!-- 등화 / 그릴 / 사이드미러 -->
-    <xacro:pair_box name="headlight" x="2.245" z="0.49"
-                    sx="0.05" sy="0.34" sz="0.14" material="valet_light" y_off="0.60"/>
-    <xacro:pair_box name="taillight" x="-2.245" z="0.55"
-                    sx="0.05" sy="0.30" sz="0.12" material="valet_tail" y_off="0.66"/>
-    <xacro:body_box name="grille" x="2.245" y="0" z="0.29"
-                    sx="0.05" sy="1.00" sz="0.16"
-                    material="valet_dark" collision="false"/>
-    <!-- 미러는 전폭 밖으로 나가므로 충돌 없음 (실차도 그렇다).
-         바깥끝 1.025 m — Nav2 footprint 반폭 1.00 + padding 0.03 안쪽 -->
-    <xacro:pair_box name="mirror" x="0.75" z="0.73"
-                    sx="0.09" sy="0.11" sz="0.07" material="valet_dark" y_off="0.97"/>
+                    material="valet_body" collision="false" visual="${not use_mesh}"/>
+    <xacro:unless value="${use_mesh}">
+      <!-- 앞유리 / 뒷유리 (기울어진 판) -->
+      <xacro:glass_panel name="windshield" x="0.60"  z="0.81" plen="0.68" pitch="0.491"/>
+      <xacro:glass_panel name="rearglass"  x="-1.085" z="0.82" plen="0.41" pitch="-0.838"/>
+      <!-- 센서 포드 (지붕 위) -->
+      <visual name="sensor_pod_vis">
+        <origin xyz="0 0 ${pod_cz}" rpy="0 0 0"/>
+        <geometry><cylinder radius="0.10" length="0.05"/></geometry>
+        <material name="valet_metal"/>
+      </visual>
+      <!-- 등화 / 그릴 / 사이드미러 -->
+      <xacro:pair_box name="headlight" x="2.245" z="0.49"
+                      sx="0.05" sy="0.34" sz="0.14" material="valet_light" y_off="0.60"/>
+      <xacro:pair_box name="taillight" x="-2.245" z="0.55"
+                      sx="0.05" sy="0.30" sz="0.12" material="valet_tail" y_off="0.66"/>
+      <xacro:body_box name="grille" x="2.245" y="0" z="0.29"
+                      sx="0.05" sy="1.00" sz="0.16"
+                      material="valet_dark" collision="false" visual="${not use_mesh}"/>
+      <!-- 미러는 전폭 밖으로 나가므로 충돌 없음 (실차도 그렇다).
+           바깥끝 1.025 m — Nav2 footprint 반폭 1.00 + padding 0.03 안쪽 -->
+      <xacro:pair_box name="mirror" x="0.75" z="0.73"
+                      sx="0.09" sy="0.11" sz="0.07" material="valet_dark" y_off="0.97"/>
+    </xacro:unless>
   </xacro:macro>
 </robot>

File: src/valet_robot/urdf/valet_car.urdf.xacro (robot description, xacro)
@@ -21,4 +21,6 @@
   <!-- 라이다를 뺀 채로 띄우고 싶을 때 (렌더링 없이 물리/제어만 검증). -->
   <xacro:arg name="lidar" default="true"/>
+  <!-- mesh:=false 면 외형이 박스 조합으로 나온다 (메시 없이 확인할 때). -->
+  <xacro:arg name="mesh" default="true"/>
   <xacro:arg name="controllers_file"
              default="$(find valet_robot)/config/controllers.yaml"/>
@@ -34,5 +36,5 @@
   </joint>
   <link name="base_link">
-    <xacro:car_body/>
+    <xacro:car_body use_mesh="$(arg mesh)"/>
     <!-- 관성: 차체 전체를 하나의 등가 박스로 근사. 무게중심은 실차처럼 낮게. -->
     <xacro:box_inertia m="${base_mass}" x="4.50" y="1.70" z="0.90">

File: src/valet_robot/urdf/wheels.xacro (robot description, xacro)
@@ -10,15 +10,25 @@
   <xacro:macro name="wheel_link" params="name">
     <link name="${name}">
-      <visual>
-        <origin xyz="0 0 0" rpy="${pi/2} 0 0"/>
-        <geometry><cylinder radius="${wheel_radius}" length="${wheel_width}"/></geometry>
-        <material name="valet_rubber"/>
-      </visual>
-      <!-- 휠(림). 타이어 안쪽에 살짝 작게 -->
-      <visual>
-        <origin xyz="0 0 0" rpy="${pi/2} 0 0"/>
-        <geometry><cylinder radius="${wheel_radius*0.62}" length="${wheel_width*1.04}"/></geometry>
-        <material name="valet_rim"/>
-      </visual>
+      <!-- 외형: 메시 (실차 타이어+휠). use_mesh 가 false 면 원통으로 대체 -->
+      <xacro:if value="$(arg mesh)">
+        <visual>
+          <origin xyz="0 0 0" rpy="0 0 0"/>
+          <geometry>
+            <mesh filename="package://valet_robot/meshes/wheel.obj"/>
+          </geometry>
+        </visual>
+      </xacro:if>
+      <xacro:unless value="$(arg mesh)">
+        <visual>
+          <origin xyz="0 0 0" rpy="${pi/2} 0 0"/>
+          <geometry><cylinder radius="${wheel_radius}" length="${wheel_width}"/></geometry>
+          <material name="valet_rubber"/>
+        </visual>
+        <visual>
+          <origin xyz="0 0 0" rpy="${pi/2} 0 0"/>
+          <geometry><cylinder radius="${wheel_radius*0.62}" length="${wheel_width*1.04}"/></geometry>
+          <material name="valet_rim"/>
+        </visual>
+      </xacro:unless>
       <collision>
         <origin xyz="0 0 0" rpy="${pi/2} 0 0"/>
@@ -33,9 +43,11 @@
     <!-- 조향 너클: 충돌 형상 없음(데크/섀시와의 자기충돌 회피) -->
     <link name="front_${side}_steer_link">
-      <visual>
-        <origin xyz="0 0 0" rpy="0 0 0"/>
-        <geometry><box size="0.12 0.09 0.24"/></geometry>
-        <material name="valet_dark"/>
-      </visual>
+      <xacro:unless value="$(arg mesh)">
+        <visual>
+          <origin xyz="0 0 0" rpy="0 0 0"/>
+          <geometry><box size="0.12 0.09 0.24"/></geometry>
+          <material name="valet_dark"/>
+        </visual>
+      </xacro:unless>
       <xacro:box_inertia m="${knuckle_mass}" x="0.14" y="0.10" z="0.26">
         <origin xyz="0 0 0" rpy="0 0 0"/>
