Commit message: valet_car: 실차 세단 형상으로 재모델링 + 조향 조인트 순서 버그 수정
## 1. 차체를 실제 승용차 형상으로 다시 만들었다

기존 저상형 플랫폼(전고 0.94 m 슬래브)에서 세단으로 교체.

  전장 4.50 x 전폭 1.90 x 전고 1.45 m  (쏘나타 1.445 / 캠리 1.455 급)
  보닛(경사판) · 캐빈 · 앞유리 · 뒷유리 · 루프 · 휠아치
  헤드램프 · 테일램프 · 그릴 · 사이드미러 · 타이어+휠 분리

하부는 축 사이(x +-0.92)에만 플로어팬을 두고 바퀴 x 구간을 비워 휠아치를
만들었다. 그 위를 전폭 벨트라인이 덮어 펜더가 된다. 앞머리는 벨트라인을
캐빈부(0.68~1.00)와 보닛부(0.68~0.94)로 나눠 낮췄다.

충돌 형상은 6개 박스로 단순하게 유지했고, 최대조향 43도 포락선까지 포함해
바퀴와 겹치지 않는 것을 check_model.py 로 검증한다.

### 라이다를 0.92 m -> 지붕 위 1.42 m 로 이동

실차 형상이면 자기 지붕(1.34)보다 위여야 360도가 안 가린다. 그 위에서
주차 차량이 존재하는 높이대는 캐빈(0.99~1.51) 하나뿐이라 1.42 m 로 잡았다.

트레이드오프: 주차 차량을 차체(4.4 m)가 아니라 캐빈(2.2 m)으로 본다.
빈 주차면 탐색에는 충분하고 통로 주행 여유(3.5 m)도 있어 실용상 문제없다.
풀 차체를 보려면 범퍼 장착(0.55 m) 전/후방 2개가 정답이지만, 이 GL 스택이
gpu_lidar 를 하나만 렌더링해서 불가능하다.

## 2. ackermann_steering_controller 조인트 순서가 [오른쪽, 왼쪽] 이었다

가장 오래 걸린 버그. traction_joints_names / steering_joints_names 를
[left, right] 로 줬더니 좌우가 뒤바뀐 Ackermann 이 걸렸다.

  좌회전(wz > 0) 인데 실측:
    좌 조향 29.9 / 우 조향 41.1   <- 우측이 내륜처럼 더 꺾임 (반대)
    좌 구동 3.62  / 우 구동 2.44   <- 우측이 내륜처럼 더 느림 (반대)

steering_controllers_library 의 SteeringOdometry::get_commands() 가
{alpha_r, alpha_l} 순으로 반환한다. 즉 index 0 이 오른쪽이다.

순서를 뒤집자 타이어 스크럽이 사라지면서

  실측 최소회전반경   4.02 m  -> 3.49 m   (요구 3.5704 이하 달성)
  각속도 추종        0.029  -> 0.251 rad/s (상한 0.280)
  좌/우 조향각       29.9/41.1 -> 39.6/30.6 (좌회전에서 좌측이 내륜)

증상이 "조향은 되는데 차가 안 돈다" 라서 좌우 조향각을 따로 찍어보기
전까지는 원인이 안 보였다.

## 3. 추가

* urdf/body.xacro          차체 형상 분리 (매크로)
* tools/preview_model.py   Gazebo 없이 URDF 만으로 4면도 PNG 생성.
                           렌더링이 막힌 환경에서 형상 확인용.
                             python3 tools/preview_model.py out.png 25
* lidar:=false 런치 인자    라이다 없이 띄워 물리/제어만 검증.
                           /dev/dri 권한이 없는 상태에서도 주행 시험 가능.
* check_model.py           바퀴 스윕 AABB 와 차체 충돌박스의 3D 겹침을
                           전수 검사하도록 강화. 라이다 높이는 차체 대역과
                           캐빈 대역 둘 다 인정하도록 수정.
* smoke_probe.py           선회 시험 코스를 Aisle_C 남쪽 시작 + 90도로 변경.
                           (최소회전반경 원의 지름 7.6 m 가 통로 폭 8 m 에
                            간신히 들어가서, 기존 14 초 선회는 주차 차량에
                            부딪혔다)

## 4. 실측 (8 항목 중 라이다 제외 7 항목, lidar:=false)

  전진 8 s @1.0 m/s     이동 8.00 m, 방향변화 0.0 deg
  최소회전반경 선회      실측 R = 3.49 m
  Ackermann 내륜차      좌 39.60 / 우 30.61 (차 8.99 deg)
  후진 5 s @-0.5 m/s    차체 전방 기준 -2.49 m
  제자리회전 차단        이동 0.000 m, 회전 0.00 deg
  각속도 클램프          요청 2.0 -> 실측 0.251, 상한 0.280
  odom -> base_footprint TF 정상

File: src/valet_robot/urdf/common.xacro (robot description, xacro)
@@ -29,29 +29,69 @@
   <xacro:property name="steer_limit"
                   value="${1.05*atan(wheelbase/(min_turn_radius - track/2))}"/>
-  <!-- ===== 2. 차체 형상 ================================================ -->
+  <!-- ===== 2. 차체 형상 (실차 세단 프로파일) ======================== -->
   <!-- base_link 는 "차체 중심"(앞뒤 오버행 각 1.00 m). 후륜축이 아니다.
        근거: nav2_ackermann.yaml footprint 가 [+-2.30, +-1.00] 대칭이고
              parking_spots.yaml 의 goal_pose 가 주차면 중심이기 때문. -->
   <xacro:property name="base_z"       value="${wheel_radius}"/>  <!-- 지면->base_link -->
-  <!-- 하부 섀시: 바퀴(안쪽끝 y=0.59)와 간섭하지 않도록 폭 1.10 -->
-  <xacro:property name="chassis_len"  value="4.20"/>
-  <xacro:property name="chassis_w"    value="1.10"/>
-  <xacro:property name="chassis_h"    value="0.42"/>
-  <xacro:property name="chassis_cz"   value="0.12"/>   <!-- base_link 기준, 절대 0.45 -->
-  <!-- 상부 데크: 전장/전폭을 담당. 바퀴 상단(절대 0.66)보다 0.02 위에서 시작 -->
-  <xacro:property name="deck_len"     value="${body_length}"/>
-  <xacro:property name="deck_w"       value="${body_width}"/>
-  <xacro:property name="deck_h"       value="0.14"/>
-  <xacro:property name="deck_cz"      value="0.42"/>   <!-- 절대 0.75, 상단 0.82 -->
+  <!-- 실차 세단 측면 프로파일 (절대 높이, m)
+         0.00          지면
+         0.24 ~ 0.66   로커/플로어팬 · 범퍼      바퀴가 드나드는 높이
+         0.68 ~ 1.00   벨트라인(펜더)            바퀴 위를 덮는 전폭 부위
+         0.98 ~ 1.06   보닛 / 트렁크 리드
+         1.02 ~ 1.30   캐빈(그린하우스) + 유리
+         1.30 ~ 1.34   루프 패널
+         1.34 ~ 1.39   센서 포드
+         1.42          라이다 스캔 평면          <- 아래 3장 참고
+       전고 1.445 m — 쏘나타(1.445) / 캠리(1.455) 급 -->
+  <!-- 하부: 바퀴가 들어갈 자리를 비워 휠아치를 만든다.
+       플로어팬은 축 사이(x +-0.92)만 전폭으로 두고, 바퀴 x 구간은 비운다.
+       최대조향(43도) 시 앞바퀴 x 는 0.934~1.566 이므로 6 cm 이상 여유. -->
+  <xacro:property name="pan_len"      value="1.84"/>   <!-- x +-0.92 -->
+  <xacro:property name="pan_w"        value="${body_width}"/>
+  <xacro:property name="pan_h"        value="0.42"/>
+  <xacro:property name="pan_cz"       value="0.12"/>   <!-- 절대 0.45 -->
+  <xacro:property name="fascia_len"   value="0.62"/>   <!-- 범퍼 블록 -->
+  <xacro:property name="fascia_w"     value="1.86"/>
+  <xacro:property name="fascia_cx"    value="1.94"/>   <!-- x 1.63~2.25 -->
+  <!-- 벨트라인: 전장/전폭을 정의하는 형상. 바퀴 상단(0.66)보다 0.02 위.
+       앞머리를 낮추려고 캐빈/후방(1.00)과 보닛부(0.94)를 나눠 놓았다. -->
+  <xacro:property name="beltr_len"    value="3.15"/>   <!-- x -2.25~0.90 -->
+  <xacro:property name="beltr_cx"     value="-0.675"/>
+  <xacro:property name="beltr_h"      value="0.32"/>
+  <xacro:property name="beltr_cz"     value="0.51"/>   <!-- 절대 0.68~1.00 -->
+  <xacro:property name="beltf_len"    value="1.35"/>   <!-- x 0.90~2.25 -->
+  <xacro:property name="beltf_cx"     value="1.575"/>
+  <xacro:property name="beltf_h"      value="0.26"/>
+  <xacro:property name="beltf_cz"     value="0.48"/>   <!-- 절대 0.68~0.94 -->
+  <!-- 보닛: 카울(0.96)에서 노즈(0.90)로 내려가는 경사판 -->
+  <xacro:property name="hood_len"     value="1.36"/>
+  <xacro:property name="hood_cx"      value="1.56"/>
+  <xacro:property name="hood_cz"      value="0.60"/>   <!-- 절대 0.93 -->
+  <xacro:property name="hood_pitch"   value="0.0441"/>
+  <xacro:property name="trunk_len"    value="1.02"/>
+  <xacro:property name="trunk_cx"     value="-1.73"/>
+  <xacro:property name="lid_w"        value="1.80"/>
+  <xacro:property name="lid_h"        value="0.08"/>
+  <xacro:property name="lid_cz"       value="0.69"/>   <!-- 절대 0.98~1.06 -->
+  <xacro:property name="cabin_len"    value="1.25"/>
+  <xacro:property name="cabin_w"      value="1.72"/>
+  <xacro:property name="cabin_h"      value="0.28"/>
+  <xacro:property name="cabin_cx"     value="-0.325"/> <!-- x -0.95~0.30 -->
+  <xacro:property name="cabin_cz"     value="0.83"/>   <!-- 절대 1.02~1.30 -->
+  <xacro:property name="roof_cz"      value="0.99"/>   <!-- 절대 1.30~1.34 -->
+  <xacro:property name="pod_cz"       value="1.035"/>  <!-- 절대 1.34~1.39 -->
   <!-- ===== 3. 센서 장착 높이 (주차장 월드 기하로부터 역산) ==============
-       parked_car 차체 박스 : z 0.27 ~ 0.99  (폭 1.80)
-       parked_car 캐빈      : z 0.99 ~ 1.51  (폭 1.66)
+       parked_car 차체 박스 : z 0.27 ~ 0.99  (폭 1.80, 길이 4.40)
+       parked_car 캐빈      : z 0.99 ~ 1.51  (폭 1.66, 길이 2.20)
        벽/기둥 2.60 · EV충전기 1.30 · 게이트 1.20 · 라바콘 0.59
-       라이다를 지붕(1.6 m)에 올리면 주차 차량 위를 넘어가 obstacle_layer 가
-       주차 차량을 못 본다. 반대로 자차 데크(0.82) 보다는 위여야 자기 몸에 가린다.
-       -> 절대 0.92 m. 주차 차량 "차체"를 때리고 자차 데크는 넘어간다.
-       라바콘(0.59)은 못 보지만 정적 맵(parking_lot.pgm)에 이미 들어있다. -->
-  <xacro:property name="lidar_z"      value="0.59"/>   <!-- 절대 0.92 -->
-  <xacro:property name="mast_cz"      value="0.52"/>   <!-- 절대 0.85 -->
+       실차 형상이면 자기 지붕(1.34)보다 위에 달아야 360도가 가려지지 않는다.
+       그러면서도 주차 차량을 봐야 하는데, 1.34 위에서 주차 차량이 있는 높이는
+       "캐빈 대역 0.99~1.51" 뿐이다. -> 1.42 m (캐빈 상단까지 9 cm 여유)
+       트레이드오프: 이 높이에서는 주차 차량이 차체(4.4 x 1.8)가 아니라
+       캐빈(2.2 x 1.66)으로 보인다. 빈 주차면 탐색에는 충분하지만 차량 외형을
+       실제보다 작게 본다. 라바콘/게이트/충전기는 못 보지만 전부 정적 맵에 있다.
+       (풀 차체를 보려면 범퍼 장착 0.55 m + FOV 제한이 필요한데, 이 GL 스택은
+        gpu_lidar 를 하나만 렌더링해서 전/후방 2개 구성이 불가능하다) -->
+  <xacro:property name="lidar_z"      value="1.09"/>   <!-- 절대 1.42 -->
   <xacro:property name="imu_z"        value="0.05"/>
   <!-- ===== 4. 질량 ===================================================== -->
@@ -83,9 +123,12 @@
   </xacro:macro>
   <!-- ===== 7. 재질 ===================================================== -->
-  <material name="valet_deck">   <color rgba="0.93 0.45 0.10 1.0"/></material>
-  <material name="valet_body">   <color rgba="0.20 0.22 0.26 1.0"/></material>
-  <material name="valet_rubber"> <color rgba="0.07 0.07 0.08 1.0"/></material>
-  <material name="valet_metal">  <color rgba="0.55 0.57 0.60 1.0"/></material>
-  <material name="valet_sensor"> <color rgba="0.10 0.60 0.85 1.0"/></material>
-  <material name="valet_front">  <color rgba="0.95 0.90 0.30 1.0"/></material>
+  <material name="valet_body">   <color rgba="0.72 0.16 0.14 1.0"/></material>  <!-- 차체색 -->
+  <material name="valet_glass">  <color rgba="0.10 0.13 0.17 0.85"/></material> <!-- 유리 -->
+  <material name="valet_dark">   <color rgba="0.07 0.07 0.08 1.0"/></material>  <!-- 그릴/미러 -->
+  <material name="valet_rubber"> <color rgba="0.06 0.06 0.07 1.0"/></material>  <!-- 타이어 -->
+  <material name="valet_rim">    <color rgba="0.72 0.74 0.78 1.0"/></material>  <!-- 휠 -->
+  <material name="valet_metal">  <color rgba="0.45 0.47 0.50 1.0"/></material>  <!-- 센서 포드 -->
+  <material name="valet_sensor"> <color rgba="0.10 0.60 0.85 1.0"/></material>  <!-- 라이다 -->
+  <material name="valet_light">  <color rgba="0.98 0.96 0.82 1.0"/></material>  <!-- 헤드램프 -->
+  <material name="valet_tail">   <color rgba="0.85 0.10 0.10 1.0"/></material>  <!-- 테일램프 -->
 </robot>

File: src/valet_robot/urdf/sensors.gazebo.xacro (robot description, xacro)
@@ -19,5 +19,5 @@
     </gazebo>
   </xacro:macro>
-  <xacro:macro name="valet_gazebo">
+  <xacro:macro name="valet_gazebo" params="lidar:=true">
     <!-- ========== 바퀴 접촉 물성 ========== -->
     <xacro:wheel_surface link="front_left_wheel_link"/>
@@ -25,36 +25,38 @@
     <xacro:wheel_surface link="rear_left_wheel_link"/>
     <xacro:wheel_surface link="rear_right_wheel_link"/>
-    <!-- ========== 2D 라이다 ==========
-         range.max 30.0 = nav2_ackermann.yaml 의 laser_max_range / raytrace_max_range
-         range.min 0.20 = laser_min_range -->
-    <gazebo reference="lidar_link">
-      <sensor name="lidar" type="gpu_lidar">
-        <topic>/scan</topic>
-        <gz_frame_id>lidar_link</gz_frame_id>
-        <update_rate>15</update_rate>
-        <always_on>true</always_on>
-        <visualize>false</visualize>
-        <lidar>
-          <scan>
-            <horizontal>
-              <samples>720</samples>
-              <resolution>1</resolution>
-              <min_angle>-3.141592</min_angle>
-              <max_angle>3.141592</max_angle>
-            </horizontal>
-          </scan>
-          <range>
-            <min>0.20</min>
-            <max>30.0</max>
-            <resolution>0.01</resolution>
-          </range>
-          <noise>
-            <type>gaussian</type>
-            <mean>0.0</mean>
-            <stddev>0.012</stddev>
-          </noise>
-        </lidar>
-      </sensor>
-    </gazebo>
+    <xacro:if value="${lidar}">
+      <!-- ========== 2D 라이다 ==========
+           range.max 30.0 = nav2_ackermann.yaml 의 laser_max_range / raytrace_max_range
+           range.min 0.20 = laser_min_range -->
+      <gazebo reference="lidar_link">
+        <sensor name="lidar" type="gpu_lidar">
+          <topic>/scan</topic>
+          <gz_frame_id>lidar_link</gz_frame_id>
+          <update_rate>15</update_rate>
+          <always_on>true</always_on>
+          <visualize>false</visualize>
+          <lidar>
+            <scan>
+              <horizontal>
+                <samples>720</samples>
+                <resolution>1</resolution>
+                <min_angle>-3.141592</min_angle>
+                <max_angle>3.141592</max_angle>
+              </horizontal>
+            </scan>
+            <range>
+              <min>0.20</min>
+              <max>30.0</max>
+              <resolution>0.01</resolution>
+            </range>
+            <noise>
+              <type>gaussian</type>
+              <mean>0.0</mean>
+              <stddev>0.012</stddev>
+            </noise>
+          </lidar>
+        </sensor>
+      </gazebo>
+    </xacro:if>
     <!-- ========== IMU ========== -->
     <gazebo reference="imu_link">

File: src/valet_robot/urdf/valet_car.urdf.xacro (robot description, xacro)
@@ -19,7 +19,10 @@
        false 면 순수 URDF (RViz 로 모델만 확인할 때). -->
   <xacro:arg name="sim" default="true"/>
+  <!-- 라이다를 뺀 채로 띄우고 싶을 때 (렌더링 없이 물리/제어만 검증). -->
+  <xacro:arg name="lidar" default="true"/>
   <xacro:arg name="controllers_file"
              default="$(find valet_robot)/config/controllers.yaml"/>
   <xacro:include filename="common.xacro"/>
+  <xacro:include filename="body.xacro"/>
   <xacro:include filename="wheels.xacro"/>
   <!-- ===================== 1. 베이스 ===================== -->
@@ -31,38 +34,8 @@
   </joint>
   <link name="base_link">
-    <!-- 하부 섀시 -->
-    <visual>
-      <origin xyz="0 0 ${chassis_cz}" rpy="0 0 0"/>
-      <geometry><box size="${chassis_len} ${chassis_w} ${chassis_h}"/></geometry>
-      <material name="valet_body"/>
-    </visual>
-    <collision>
-      <origin xyz="0 0 ${chassis_cz}" rpy="0 0 0"/>
-      <geometry><box size="${chassis_len} ${chassis_w} ${chassis_h}"/></geometry>
-    </collision>
-    <!-- 상부 데크 — 전장 4.50 x 전폭 1.90 을 정의하는 형상 -->
-    <visual>
-      <origin xyz="0 0 ${deck_cz}" rpy="0 0 0"/>
-      <geometry><box size="${deck_len} ${deck_w} ${deck_h}"/></geometry>
-      <material name="valet_deck"/>
-    </visual>
-    <collision>
-      <origin xyz="0 0 ${deck_cz}" rpy="0 0 0"/>
-      <geometry><box size="${deck_len} ${deck_w} ${deck_h}"/></geometry>
-    </collision>
-    <!-- 앞머리 식별 마커 (충돌 없음) -->
-    <visual>
-      <origin xyz="${deck_len/2.0 - 0.06} 0 ${deck_cz + deck_h/2.0 + 0.02}" rpy="0 0 0"/>
-      <geometry><box size="0.12 ${deck_w*0.75} 0.05"/></geometry>
-      <material name="valet_front"/>
-    </visual>
-    <!-- 센서 마스트 (충돌 없음) -->
-    <visual>
-      <origin xyz="0 0 ${mast_cz}" rpy="0 0 0"/>
-      <geometry><cylinder radius="0.05" length="0.06"/></geometry>
-      <material name="valet_metal"/>
-    </visual>
-    <xacro:box_inertia m="${base_mass}" x="4.50" y="1.60" z="0.60">
-      <origin xyz="0 0 0.22" rpy="0 0 0"/>
+    <xacro:car_body/>
+    <!-- 관성: 차체 전체를 하나의 등가 박스로 근사. 무게중심은 실차처럼 낮게. -->
+    <xacro:box_inertia m="${base_mass}" x="4.50" y="1.70" z="0.90">
+      <origin xyz="-0.05 0 0.22" rpy="0 0 0"/>
     </xacro:box_inertia>
   </link>
@@ -81,22 +54,24 @@
   <xacro:rear_corner  side="right" reflect="-1"/>
   <!-- ===================== 3. 센서 프레임 ===================== -->
-  <!-- 2D 라이다 — 절대 높이 0.92 m (근거는 common.xacro 주석) -->
-  <link name="lidar_link">
-    <visual>
-      <origin xyz="0 0 0" rpy="0 0 0"/>
-      <geometry><cylinder radius="0.055" length="0.07"/></geometry>
-      <material name="valet_sensor"/>
-    </visual>
-    <inertial>
-      <origin xyz="0 0 0" rpy="0 0 0"/>
-      <mass value="1.2"/>
-      <inertia ixx="0.002" ixy="0" ixz="0" iyy="0.002" iyz="0" izz="0.002"/>
-    </inertial>
-  </link>
-  <joint name="lidar_joint" type="fixed">
-    <parent link="base_link"/>
-    <child  link="lidar_link"/>
-    <origin xyz="0 0 ${lidar_z}" rpy="0 0 0"/>
-  </joint>
+  <!-- 2D 라이다 — 지붕 위 절대 높이 1.42 m (근거는 common.xacro 3장) -->
+  <xacro:if value="$(arg lidar)">
+    <link name="lidar_link">
+      <visual>
+        <origin xyz="0 0 0" rpy="0 0 0"/>
+        <geometry><cylinder radius="0.055" length="0.05"/></geometry>
+        <material name="valet_sensor"/>
+      </visual>
+      <inertial>
+        <origin xyz="0 0 0" rpy="0 0 0"/>
+        <mass value="1.2"/>
+        <inertia ixx="0.002" ixy="0" ixz="0" iyy="0.002" iyz="0" izz="0.002"/>
+      </inertial>
+    </link>
+    <joint name="lidar_joint" type="fixed">
+      <parent link="base_link"/>
+      <child  link="lidar_link"/>
+      <origin xyz="0 0 ${lidar_z}" rpy="0 0 0"/>
+    </joint>
+  </xacro:if>
   <link name="imu_link">
     <inertial>
@@ -116,5 +91,5 @@
     <xacro:include filename="sensors.gazebo.xacro"/>
     <xacro:valet_ros2_control controllers_file="$(arg controllers_file)"/>
-    <xacro:valet_gazebo/>
+    <xacro:valet_gazebo lidar="$(arg lidar)"/>
   </xacro:if>
 </robot>

File: src/valet_robot/urdf/wheels.xacro (robot description, xacro)
@@ -15,9 +15,9 @@
         <material name="valet_rubber"/>
       </visual>
-      <!-- 휠 디스크 (방향 식별용, 충돌 없음) -->
+      <!-- 휠(림). 타이어 안쪽에 살짝 작게 -->
       <visual>
         <origin xyz="0 0 0" rpy="${pi/2} 0 0"/>
-        <geometry><cylinder radius="${wheel_radius*0.55}" length="${wheel_width*1.06}"/></geometry>
-        <material name="valet_metal"/>
+        <geometry><cylinder radius="${wheel_radius*0.62}" length="${wheel_width*1.04}"/></geometry>
+        <material name="valet_rim"/>
       </visual>
       <collision>
@@ -35,6 +35,6 @@
       <visual>
         <origin xyz="0 0 0" rpy="0 0 0"/>
-        <geometry><box size="0.14 0.10 0.26"/></geometry>
-        <material name="valet_metal"/>
+        <geometry><box size="0.12 0.09 0.24"/></geometry>
+        <material name="valet_dark"/>
       </visual>
       <xacro:box_inertia m="${knuckle_mass}" x="0.14" y="0.10" z="0.26">
