Commit message: 전방 하향 RGBD 카메라 추가 — 라이다 사각(1.42 m 아래) 을 코스트맵에 연결
판단 근거가 2D 라이다 한 평면뿐이었다. 절대 1.42 m 에서만 보므로 그 아래
물체는 존재하지 않는 것과 같다. 실측으로 4 m 앞 트래픽 콘(높이 0.55 m)에
대해 라이다는 전방 +-14 도 최소거리 8.13 m 를 반환했다. 아예 못 본다.
지금 콘을 피하는 건 센서가 아니라 정적 맵에 미리 칠해 둔 덕이고
(generate_parking_lot.py 의 fill_box(..., OCC)) 런타임에 생기는 낮은
장애물에는 무방비다.

앞면 그릴 높이(절대 0.95 m)에 하향 20 도로 RGBD 를 달고, 포인트클라우드를
전역/지역 코스트맵의 obstacle_layer 관측원으로 넣었다.

## 검증

같은 자세에서 카메라는 콘을 3742 점으로 잡았고 범위가 실물과 일치했다.

    카메라가 본 콘  x -6.22~-5.79  y -22.31~-21.87  z 0.10~0.55
    실제 콘         중심 (-6.0,-22.05) 반지름 0.22 높이 0.55

정적 맵에 없는 자리로 콘을 옮기고 같은 목표로 주행시켰다.

    콘 있음   x -0.53 -> y -16.48    최근접 2.40 m,  status 4 (성공)
    대조군    x -0.13 -> y -19.05
                                     2.5 m 북쪽으로 우회

주차 정확도는 그대로다 (A08 0.08 m / B05 0.03 m, 변경 전 0.02~0.08 m).

## 데인 곳

1) gz 의 rgbd_camera 는 점을 x=전방 / y=좌 / z=상 으로 낸다. ROS 카메라
   규약(z=전방)이 아니다. frame_id 에 광학 프레임 이름을 찍으면 TF 가
   회전을 한 번 더 걸어서 구름이 통째로 눕는다 (지면 점이 z -8 m 로
   내려가고 콘이 사라졌다). gz_frame_id 는 camera_link 여야 한다.
   원시 좌표의 x 가 1.14~14.06 인 것으로 축을 확인했다.

2) optical_frame_id 를 쓰면 안 된다. 그게 포인트클라우드의 frame_id 까지
   덮어써서 gz_frame_id 가 무시된다.

3) min_obstacle_height 는 필수다. 하향 카메라라 구름의 78 % (67013 중
   52196 점) 가 지면이다. 없으면 바닥을 장애물로 찍는다.
   (다행히 시뮬 지면은 깨끗했다 — 전 거리대에서 z 중앙값 -0.000,
    최대 +0.020, 0.12 초과 0.0 %.)

4) 보닛 위에 달면 안 된다. 보닛 상면이 절대 1.06 이라 (x 2.10, z 1.10) 에
   두면 보닛 앞모서리가 수평 아래 15 도에 걸려 그보다 가파른 시선이
   전부 막힌다.

## 시험할 때 주의

콘을 gz set_pose 로 옮겨도 정적 맵에는 옛 자리가 그대로 남는다. 그래서
장애물이 둘이 되고, 두 내접 대역(각 +-1.03 m)이 엇갈리면 8 m 통로가
통째로 끊긴다. 실제로 그렇게 만들어 놓고 "회피 실패" 로 오인했는데
코스트맵을 떠 보니 플래너가 맞았다. 새 장애물은 원래 자리에서 충분히
떨어뜨릴 것.

해상도/주기를 올리지 말 것. 320x240 @ 10 Hz 도 소프트웨어 렌더링에서는
6~8 Hz 밖에 안 나온다. camera:=false 로 뺄 수 있다.

File: src/valet_robot/urdf/common.xacro (robot description, xacro)
@@ -81,4 +81,17 @@
   <xacro:property name="roof_cz"      value="0.99"/>   <!-- 절대 1.30~1.34 -->
   <xacro:property name="pod_cz"       value="1.035"/>  <!-- 절대 1.34~1.39 -->
+  <!-- 전방 하향 RGBD 카메라 — 앞면 그릴 높이(절대 0.95 m)에 앞면보다
+       3 cm 앞으로 내민다. 2D 라이다 평면(1.42 m) 아래를 덮는 게 목적이다.
+       월드의 트래픽 콘은 높이 0.55 m 라 라이다로는 아예 안 보인다.
+       ! 보닛 위에 달면 안 된다. 보닛 상면이 절대 1.06 이라 카메라를
+         (x 2.10, z 1.10) 에 두면 보닛 앞모서리 (2.25, 1.06) 이 수평
+         아래 15 도에 걸려서 그보다 가파른 시선이 전부 막힌다.
+         그릴 높이면 앞이 트여 있다.
+       하향 20 도 + vFOV 55.4 도(hFOV 70, 4:3) 이므로 시야 하단이
+       47.7 도. 지면을 0.95/tan(47.7) = 0.86 m 앞에서 잡기 시작한다
+       (범퍼 기준 0.89 m 사각). 4.5 m 차량으로선 정상 범위. -->
+  <xacro:property name="cam_x"     value="2.28"/>
+  <xacro:property name="cam_z"     value="0.62"/>   <!-- 절대 0.95 -->
+  <xacro:property name="cam_pitch" value="0.3491"/> <!-- 하향 20 deg -->
   <!-- ===== 3. 센서 장착 높이 (주차장 월드 기하로부터 역산) ==============
        parked_car 차체 박스 : z 0.27 ~ 0.99  (폭 1.80, 길이 4.40)

File: src/valet_robot/urdf/sensors.gazebo.xacro (robot description, xacro)
@@ -4,4 +4,6 @@
      발행 토픽 (gz)      -> ros_gz_bridge 로 ROS 2 에 넘어감
        /scan             sensor_msgs/LaserScan   (AMCL, costmap obstacle_layer)
+       /front_cam/image  sensor_msgs/Image
+       /front_cam/points sensor_msgs/PointCloud2 (costmap obstacle_layer)
        /imu              sensor_msgs/Imu
        /odom             nav_msgs/Odometry       (odom -> base_footprint)
@@ -19,5 +21,5 @@
     </gazebo>
   </xacro:macro>
-  <xacro:macro name="valet_gazebo" params="lidar:=true">
+  <xacro:macro name="valet_gazebo" params="lidar:=true camera:=true">
     <!-- ========== 바퀴 접촉 물성 ========== -->
     <xacro:wheel_surface link="front_left_wheel_link"/>
@@ -59,4 +61,44 @@
       </gazebo>
     </xacro:if>
+    <xacro:if value="${camera}">
+      <!-- ========== 전방 하향 RGBD ==========
+           2D 라이다는 절대 1.42 m 한 평면만 본다. 그 아래는 전부 사각이라
+           월드의 트래픽 콘(높이 0.55 m)조차 안 보인다. 지금 콘을 피하는 건
+           센서가 아니라 정적 맵에 미리 칠해 둔 덕이다
+           (generate_parking_lot.py 의 fill_box(..., OCC)).
+           런타임에 생기는 낮은 장애물은 못 본다. 그걸 이 카메라가 덮는다.
+           ! 해상도와 주기를 올리지 말 것. 소프트웨어 렌더링이라 비싸다.
+             320x240 @ 10 Hz 에서 포인트가 초당 768k 나온다. 이미 GUI 만
+             켜도 3 코어를 먹는 VM 이다. -->
+      <gazebo reference="camera_link">
+        <sensor name="front_cam" type="rgbd_camera">
+          <topic>front_cam</topic>
+          <!-- ! 포인트클라우드의 frame_id 는 camera_link(차체 규약) 여야 한다.
+               gz 의 rgbd_camera 는 점을 x=전방 / y=좌 / z=상 으로 낸다.
+               ROS 카메라 규약(z=전방)이 아니다. 여기에 광학 프레임 이름을
+               찍으면 TF 가 회전을 한 번 더 걸어서 구름이 통째로 눕는다.
+               (실측: 지면 점이 z -8 m 로 내려가고 콘이 사라졌다.
+                원시 좌표의 x 가 1.14~14.06 인 것으로 확인 — 깊이 축이 x 다.)
+               optical_frame_id 를 쓰면 안 된다. 그게 포인트클라우드의
+               frame_id 까지 덮어써서 gz_frame_id 가 무시된다 (실측). -->
+          <gz_frame_id>camera_link</gz_frame_id>
+          <update_rate>10</update_rate>
+          <always_on>true</always_on>
+          <visualize>false</visualize>
+          <camera>
+            <horizontal_fov>1.2217</horizontal_fov>   <!-- 70 deg -->
+            <image>
+              <width>320</width>
+              <height>240</height>
+              <format>R8G8B8</format>
+            </image>
+            <clip>
+              <near>0.3</near>
+              <far>15.0</far>
+            </clip>
+          </camera>
+        </sensor>
+      </gazebo>
+    </xacro:if>
     <!-- ========== IMU ========== -->
     <gazebo reference="imu_link">

File: src/valet_robot/urdf/valet_car.urdf.xacro (robot description, xacro)
@@ -22,4 +22,6 @@
   <xacro:arg name="lidar" default="true"/>
   <!-- mesh:=false 면 외형이 박스 조합으로 나온다 (메시 없이 확인할 때). -->
+  <!-- 전방 RGBD 카메라. 렌더링 부하가 커서 끌 수 있게 둔다. -->
+  <xacro:arg name="camera" default="true"/>
   <xacro:arg name="mesh" default="true"/>
   <xacro:arg name="controllers_file"
@@ -76,4 +78,33 @@
     </joint>
   </xacro:if>
+  <!-- 전방 하향 RGBD (치수 근거는 common.xacro) -->
+  <xacro:if value="$(arg camera)">
+    <link name="camera_link">
+      <visual>
+        <origin xyz="0 0 0" rpy="0 0 0"/>
+        <geometry><box size="0.04 0.10 0.04"/></geometry>
+        <material name="valet_sensor"/>
+      </visual>
+      <inertial>
+        <origin xyz="0 0 0" rpy="0 0 0"/>
+        <mass value="0.15"/>
+        <inertia ixx="1e-4" ixy="0" ixz="0" iyy="1e-4" iyz="0" izz="1e-4"/>
+      </inertial>
+    </link>
+    <joint name="camera_joint" type="fixed">
+      <parent link="base_link"/>
+      <child  link="camera_link"/>
+      <origin xyz="${cam_x} 0 ${cam_z}" rpy="0 ${cam_pitch} 0"/>
+    </joint>
+    <!-- ! 광학 프레임을 따로 둔다. ROS 의 카메라 규약은 z 가 앞,
+         x 가 오른쪽, y 가 아래인데 URDF 링크는 x 가 앞이다. 이걸 안 맞추면
+         포인트클라우드가 90 도 누워서 코스트맵에 엉뚱하게 찍힌다. -->
+    <link name="camera_optical_link"/>
+    <joint name="camera_optical_joint" type="fixed">
+      <parent link="camera_link"/>
+      <child  link="camera_optical_link"/>
+      <origin xyz="0 0 0" rpy="${-pi/2} 0 ${-pi/2}"/>
+    </joint>
+  </xacro:if>
   <link name="imu_link">
     <inertial>
@@ -93,5 +124,5 @@
     <xacro:include filename="sensors.gazebo.xacro"/>
     <xacro:valet_ros2_control controllers_file="$(arg controllers_file)"/>
-    <xacro:valet_gazebo lidar="$(arg lidar)"/>
+    <xacro:valet_gazebo lidar="$(arg lidar)" camera="$(arg camera)"/>
   </xacro:if>
 </robot>
